File: 2023KicadLibrary-main/Standardized Subsheets/LDO.kicad_sch (KiCad schematic)
At the start: 3 parts

Commit message: with layout
Parts:
- gave numbers to parts that had none: 3
Changed lines of the file:
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@@
   (symbol (lib_id "power:GND") (at 96.52 91.44 0) (unit 1)
     (in_bom yes) (on_board yes) (fields_autoplaced)
-    (property "Reference" "#PWR?" (id 0) (at 96.52 97.79 0)
+    (property "Reference" "#PWR079" (id 0) (at 96.52 97.79 0)
       (effects (font (size 1.27 1.27)) hide)
     )
@@
   (symbol (lib_id "Device:C") (at 123.19 87.63 0) (unit 1)
     (in_bom yes) (on_board yes) (fields_autoplaced)
-    (property "Reference" "C?" (id 0) (at 127 86.3599 0)
+    (property "Reference" "C36" (id 0) (at 127 86.3599 0)
       (effects (font (size 1.27 1.27)) (justify left))
     )
@@
   (symbol (lib_id "power:GND") (at 111.76 91.44 0) (unit 1)
     (in_bom yes) (on_board yes) (fields_autoplaced)
-    (property "Reference" "#PWR?" (id 0) (at 111.76 97.79 0)
+    (property "Reference" "#PWR080" (id 0) (at 111.76 97.79 0)
       (effects (font (size 1.27 1.27)) hide)
     )
@@
   (symbol (lib_id "power:GND") (at 123.19 91.44 0) (unit 1)
     (in_bom yes) (on_board yes) (fields_autoplaced)
-    (property "Reference" "#PWR?" (id 0) (at 123.19 97.79 0)
+    (property "Reference" "#PWR081" (id 0) (at 123.19 97.79 0)
       (effects (font (size 1.27 1.27)) hide)
     )
@@
   (symbol (lib_id "Device:C") (at 96.52 87.63 0) (unit 1)
     (in_bom yes) (on_board yes) (fields_autoplaced)
-    (property "Reference" "C?" (id 0) (at 100.33 86.3599 0)
+    (property "Reference" "C35" (id 0) (at 100.33 86.3599 0)
       (effects (font (size 1.27 1.27)) (justify left))
     )
@@
   (symbol (lib_id "Regulator_Linear:AMS1117-3.3") (at 111.76 83.82 0) (unit 1)
     (in_bom yes) (on_board yes) (fields_autoplaced)
-    (property "Reference" "U?" (id 0) (at 111.76 76.2 0))
+    (property "Reference" "U6" (id 0) (at 111.76 76.2 0))
     (property "Value" "~" (id 1) (at 111.76 78.74 0))
     (property "Footprint" "" (id 2) (at 111.76 78.74 0)
