File: 2023KicadLibrary-main/Standardized Subsheets/BUCK.kicad_sch (KiCad schematic)
At the start: 11 parts

Commit message: with layout
Parts:
- gave numbers to parts that had none: 11
Changed lines of the file:
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@@
   (symbol (lib_id "Device:C") (at 199.39 78.105 0) (unit 1)
     (in_bom yes) (on_board yes) (fields_autoplaced)
-    (property "Reference" "C?" (id 0) (at 203.2 76.8349 0)
+    (property "Reference" "C34" (id 0) (at 203.2 76.8349 0)
       (effects (font (size 1.27 1.27)) (justify left))
     )
@@
   (symbol (lib_id "power:GND") (at 193.04 81.915 0) (unit 1)
     (in_bom yes) (on_board yes) (fields_autoplaced)
-    (property "Reference" "#PWR?" (id 0) (at 193.04 88.265 0)
+    (property "Reference" "#PWR078" (id 0) (at 193.04 88.265 0)
       (effects (font (size 1.27 1.27)) hide)
     )
@@
   (symbol (lib_id "Device:C") (at 185.42 78.105 0) (unit 1)
     (in_bom yes) (on_board yes) (fields_autoplaced)
-    (property "Reference" "C?" (id 0) (at 189.23 76.8349 0)
+    (property "Reference" "C33" (id 0) (at 189.23 76.8349 0)
       (effects (font (size 1.27 1.27)) (justify left))
     )
@@
   (symbol (lib_id "Device:C") (at 92.71 83.185 0) (unit 1)
     (in_bom yes) (on_board yes) (fields_autoplaced)
-    (property "Reference" "C?" (id 0) (at 96.52 81.9149 0)
+    (property "Reference" "C29" (id 0) (at 96.52 81.9149 0)
       (effects (font (size 1.27 1.27)) (justify left))
     )
@@
   (symbol (lib_id "Device:C") (at 104.14 83.185 0) (unit 1)
     (in_bom yes) (on_board yes) (fields_autoplaced)
-    (property "Reference" "C?" (id 0) (at 107.95 81.9149 0)
+    (property "Reference" "C30" (id 0) (at 107.95 81.9149 0)
       (effects (font (size 1.27 1.27)) (justify left))
     )
@@
   (symbol (lib_id "Device:C") (at 115.57 83.185 0) (unit 1)
     (in_bom yes) (on_board yes) (fields_autoplaced)
-    (property "Reference" "C?" (id 0) (at 119.38 81.9149 0)
+    (property "Reference" "C31" (id 0) (at 119.38 81.9149 0)
       (effects (font (size 1.27 1.27)) (justify left))
     )
@@
   (symbol (lib_id "power:GND") (at 143.51 89.535 0) (unit 1)
     (in_bom yes) (on_board yes) (fields_autoplaced)
-    (property "Reference" "#PWR?" (id 0) (at 143.51 95.885 0)
+    (property "Reference" "#PWR076" (id 0) (at 143.51 95.885 0)
       (effects (font (size 1.27 1.27)) hide)
     )
@@
   (symbol (lib_id "Device:R") (at 170.18 84.455 90) (unit 1)
     (in_bom yes) (on_board yes)
-    (property "Reference" "R?" (id 0) (at 170.18 86.995 90))
+    (property "Reference" "R43" (id 0) (at 170.18 86.995 90))
     (property "Value" "~" (id 1) (at 170.18 89.535 90))
     (property "Footprint" "" (id 2) (at 170.18 86.233 90)
@@
   (symbol (lib_id "Device:R") (at 127 83.185 0) (unit 1)
     (in_bom yes) (on_board yes) (fields_autoplaced)
-    (property "Reference" "R?" (id 0) (at 129.54 81.9149 0)
+    (property "Reference" "R41" (id 0) (at 129.54 81.9149 0)
       (effects (font (size 1.27 1.27)) (justify left))
     )
@@
   (symbol (lib_id "power:GND") (at 158.75 92.075 0) (unit 1)
     (in_bom yes) (on_board yes) (fields_autoplaced)
-    (property "Reference" "#PWR?" (id 0) (at 158.75 98.425 0)
+    (property "Reference" "#PWR077" (id 0) (at 158.75 98.425 0)
       (effects (font (size 1.27 1.27)) hide)
     )
@@
   (symbol (lib_id "Regulator_Switching:TPS562200") (at 143.51 81.915 0) (unit 1)
     (in_bom yes) (on_board yes) (fields_autoplaced)
-    (property "Reference" "U?" (id 0) (at 143.51 71.755 0))
+    (property "Reference" "U5" (id 0) (at 143.51 71.755 0))
     (property "Value" "~" (id 1) (at 143.51 74.295 0))
     (property "Footprint" "" (id 2) (at 144.78 88.265 0)
@@
   (symbol (lib_id "Device:C") (at 160.02 78.105 0) (unit 1)
     (in_bom yes) (on_board yes) (fields_autoplaced)
-    (property "Reference" "C?" (id 0) (at 163.83 76.8349 0)
+    (property "Reference" "C32" (id 0) (at 163.83 76.8349 0)
       (effects (font (size 1.27 1.27)) (justify left))
     )
@@
   (symbol (lib_id "Device:R") (at 158.75 88.265 0) (unit 1)
     (in_bom yes) (on_board yes) (fields_autoplaced)
-    (property "Reference" "R?" (id 0) (at 161.29 86.9949 0)
+    (property "Reference" "R42" (id 0) (at 161.29 86.9949 0)
       (effects (font (size 1.27 1.27)) (justify left))
     )
@@
   (symbol (lib_id "power:PWR_FLAG") (at 96.52 78.74 0) (unit 1)
     (in_bom yes) (on_board yes) (fields_autoplaced)
-    (property "Reference" "#FLG?" (id 0) (at 96.52 76.835 0)
+    (property "Reference" "#FLG05" (id 0) (at 96.52 76.835 0)
       (effects (font (size 1.27 1.27)) hide)
     )
@@
   (symbol (lib_id "Device:L") (at 173.99 74.295 90) (unit 1)
     (in_bom yes) (on_board yes) (fields_autoplaced)
-    (property "Reference" "L?" (id 0) (at 173.99 67.945 90))
+    (property "Reference" "L3" (id 0) (at 173.99 67.945 90))
     (property "Value" "~" (id 1) (at 173.99 70.485 90))
     (property "Footprint" "" (id 2) (at 173.99 74.295 0)
@@
   (symbol (lib_id "power:GND") (at 104.14 92.075 0) (unit 1)
     (in_bom yes) (on_board yes) (fields_autoplaced)
-    (property "Reference" "#PWR?" (id 0) (at 104.14 98.425 0)
-      (effects (font (size 1.27 1.27)) hide)
-    )
+    (property "Reference" "#PWR075" (id 0) (at 104.14 98.425 0)
+      (effects (font (size 1.27 1.27)) hide)
+    )
