File: 2023KicadLibrary-main/Standardized Subsheets/SEPIC_CAD.kicad_sch (KiCad schematic)
At the start: 25 parts, among them IC1 LM5155DSSR, Q1 CSD18537NQ5A

Commit message: with layout
Parts:
- renumbered C1 to C17, C2 to C18, C3 to C19, C4 to C20, C5 to C21, C6 to C22, C7 to C23, C8 to C24, C9 to C25, C10 to C26, C11 to C27, C12 to C28, D1 to D10, L1 to L2, R1 to R32, R2 to R33, R3 to R34, R4 to R35, R5 to R36, R6 to R37, R7 to R38, R8 to R39, R9 to R40

Commit message: new HUD PCB
Parts:
- C17, C18, C19, C20, C21, C22, C23, C24, C25, C26, C27, C28: footprint (none) -> Capacitor_SMD:C_0603_1608Metric
- D10: footprint D2PAK_STM -> Global Libraries_2:STPS20M100SG-TR
- L2: footprint (none) -> Inductor Thing:WE-DD_12XX_CROSSED12
- R32, R33, R34, R35, R36, R37, R38, R39, R40: footprint (none) -> Resistor_SMD:R_0603_1608Metric
