File: 2023KicadLibrary-main/Standardized Subsheets/vrmsv2.kicad_sch (KiCad schematic)
At the start: 5 parts

Commit message: with layout
Parts:
- renumbered R23 to R12
Changed lines of the file:
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@@
   (symbol (lib_id "power:+3V3") (at 151.13 36.83 0) (unit 1)
     (in_bom yes) (on_board yes) (fields_autoplaced)
-    (property "Reference" "#PWR?" (id 0) (at 151.13 40.64 0)
+    (property "Reference" "#PWR021" (id 0) (at 151.13 40.64 0)
       (effects (font (size 1.27 1.27)) hide)
     )
@@
   (symbol (lib_id "power:+5V") (at 115.57 36.83 0) (unit 1)
     (in_bom yes) (on_board yes) (fields_autoplaced)
-    (property "Reference" "#PWR?" (id 0) (at 115.57 40.64 0)
+    (property "Reference" "#PWR020" (id 0) (at 115.57 40.64 0)
       (effects (font (size 1.27 1.27)) hide)
     )
@@
   (symbol (lib_id "power:GND") (at 68.58 54.61 0) (unit 1)
     (in_bom yes) (on_board yes) (fields_autoplaced)
-    (property "Reference" "#PWR?" (id 0) (at 68.58 60.96 0)
+    (property "Reference" "#PWR018" (id 0) (at 68.58 60.96 0)
       (effects (font (size 1.27 1.27)) hide)
     )
@@
   (symbol (lib_id "power:+24V") (at 49.53 45.72 0) (unit 1)
     (in_bom yes) (on_board yes) (fields_autoplaced)
-    (property "Reference" "#PWR?" (id 0) (at 49.53 49.53 0)
+    (property "Reference" "#PWR017" (id 0) (at 49.53 49.53 0)
       (effects (font (size 1.27 1.27)) hide)
     )
@@
   (symbol (lib_id "Device:R") (at 83.82 60.96 180) (unit 1)
     (in_bom yes) (on_board yes)
-    (property "Reference" "R23" (id 0) (at 86.36 60.96 90))
+    (property "Reference" "R12" (id 0) (at 86.36 60.96 90))
     (property "Value" "470R" (id 1) (at 88.9 60.96 90))
     (property "Footprint" "Resistor_SMD:R_0603_1608Metric_Pad0.98x0.95mm_HandSolder" (id 2) (at 85.598 60.96 90)
@@
   (symbol (lib_id "power:GND") (at 83.82 64.77 0) (unit 1)
     (in_bom yes) (on_board yes) (fields_autoplaced)
-    (property "Reference" "#PWR?" (id 0) (at 83.82 71.12 0)
+    (property "Reference" "#PWR019" (id 0) (at 83.82 71.12 0)
       (effects (font (size 1.27 1.27)) hide)
     )

Commit message: new HUD PCB
Other:
- sheet BUCK: file BUCK.kicad_sch -> ../../../../Downloads/2023KicadLibrary-main 2/Standardized Subsheets/BUCK.kicad_sch
- sheet LDO: file LDO.kicad_sch -> ../../../../Downloads/2023KicadLibrary-main 2/Standardized Subsheets/LDO.kicad_sch
Changed lines of the file:
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@@
       (effects (font (size 1.27 1.27)) (justify left bottom))
     )
-    (property "Sheet file" "BUCK.kicad_sch" (id 1) (at 88.9 50.1146 0)
-      (effects (font (size 1.27 1.27)) (justify left top))
+    (property "Sheet file" "../../../../Downloads/2023KicadLibrary-main 2/Standardized Subsheets/BUCK.kicad_sch" (id 1) (at 88.9 50.1146 0)
+      (effects (font (size 1.27 1.27)) (justify left top) hide)
     )
     (pin "V_in" input (at 88.9 45.72 180)
@@
       (effects (font (size 1.27 1.27)) (justify left bottom))
     )
-    (property "Sheet file" "LDO.kicad_sch" (id 1) (at 121.92 50.7496 0)
-      (effects (font (size 1.27 1.27)) (justify left top))
+    (property "Sheet file" "../../../../Downloads/2023KicadLibrary-main 2/Standardized Subsheets/LDO.kicad_sch" (id 1) (at 121.92 50.7496 0)
+      (effects (font (size 1.27 1.27)) (justify left top) hide)
     )
     (pin "V_in" input (at 121.92 45.72 180)
