File: Charging_Case_HUD/Charging_Case_HUD.kicad_pcb (KiCad board)
At the start: 2 copper layers, 77 x 113 mm, 111 parts, among them J1 Conn_01x20, J2 09551296822741, J3 Conn_01x02, J4 Conn_01x02, J5 Conn_01x02, J6 Conn_01x02, J7 Conn_01x02, J8 SWD, SW1 SW_DIP_x01, SW2 SW_MEC_5G, SW3 SW_DIP_x01, SW4 SW_SPDT, U1 ILI9163C, U2 STM32F105RCTx, U3 SN65HVD230, U4 SN65HVD230, U5 TPS562200, U6 AMS1117-3.3, Y1 16MHz

Commit message: try 1
Parts:
- removed C17, C18: 10uF, Capacitor_SMD:C_0603_1608Metric_Pad1.08x0.95mm_HandSolder
- removed C19, C20: 100nF, Capacitor_SMD:C_0603_1608Metric_Pad1.08x0.95mm_HandSolder
- removed C21, C22, C24: 22uF, Capacitor_SMD:C_0603_1608Metric_Pad1.08x0.95mm_HandSolder
- removed C23: 1uF, Capacitor_SMD:C_0603_1608Metric_Pad1.08x0.95mm_HandSolder
- removed D8: SMLVN6RGB, LED_SMD:LED_ROHM_SMLVN6
- removed L2: 4u7, Inductor_SMD:L_Sunlord_MWSA0518_5.4x5.2mm
- removed PWR_3V1, PWR_IN1, PWR_IN2: LED, LED_SMD:LED_0603_1608Metric_Pad1.05x0.95mm_HandSolder
- removed PWR_5V1: 100, Resistor_SMD:R_0201_0603Metric_Pad0.64x0.40mm_HandSolder
- removed R32: 22, Resistor_SMD:R_0603_1608Metric
- removed R33, R34: 10K, Resistor_SMD:R_0603_1608Metric_Pad0.98x0.95mm_HandSolder
- removed R35: 54.9K, Resistor_SMD:R_0603_1608Metric_Pad0.98x0.95mm_HandSolder
- removed SW4: SW_SPDT, Connector_PinHeader_1.27mm:PinHeader_1x03_P1.27mm_Vertical
- removed U5: TPS562200, Package_TO_SOT_SMD:SOT-23-6
- removed U6: AMS1117-3.3, Package_TO_SOT_SMD:SOT-223-3_TabPin2
- added D9: SMLVN6RGB, LED_SMD:LED_ROHM_SMLVN6, F.Cu at (85.5, 176.9)
- added S1: 465031772505, Button Switch:465031772505, F.Cu at (94.0, 36.0)
- D1: footprint LED_SMD:LED_0805_2012Metric -> Dashboard_LED:LEDC1608X80N
- D4: value 20V -> 32V; footprint Diode_SMD:D_0603_1608Metric_Pad1.05x0.95mm_HandSolder -> Diode_SMD:D_SOD-323
- D5: footprint Diode_SMD:D_0603_1608Metric_Pad1.05x0.95mm_HandSolder -> Diode_SMD:D_SMA
- D6: value RED -> LED; footprint LED_SMD:LED_0603_1608Metric -> LED_SMD:LED_0603_1608Metric_Pad1.05x0.95mm_HandSolder
- D7: value DT1446-04TS-7 -> RED; footprint Global Libraries:SOT95P280X100-6N -> LED_SMD:LED_0603_1608Metric
- F1: footprint Fuse:Fuse_0603_1608Metric_Pad1.05x0.95mm_HandSolder -> Fuse:Fuse_1206_3216Metric_Pad1.42x1.75mm_HandSolder
- J1: footprint Connector_Pin:Pin_D1.3mm_L11.0mm -> Connector_PinHeader_2.54mm:PinHeader_1x20_P2.54mm_Vertical
- R1, R2: value 220 -> 150
- R12: value 470 -> 470R; footprint Resistor_SMD:R_0201_0603Metric_Pad0.64x0.40mm_HandSolder -> Resistor_SMD:R_0603_1608Metric_Pad0.98x0.95mm_HandSolder
- R13: value 0 -> 2k2; footprint Resistor_SMD:R_0201_0603Metric_Pad0.64x0.40mm_HandSolder -> Resistor_SMD:R_0603_1608Metric
- R17: value 2k2 -> 100
- R18: value 100 -> 220
- R21: value 220 -> 120
- R29: value 120 -> 47
- R3: value 200 -> 500
- R30: value 47 -> 10K
- R31: value 10K -> 22
- SW1: value SW_DIP_x01 -> SW_MEC_5G; footprint Connector:Banana_Jack_2Pin -> Button_Switch_SMD:SW_SPST_SKQG_WithStem
- SW2: value SW_MEC_5G -> SW_DIP_x01; footprint Button_Switch_SMD:SW_SPST_SKQG_WithStem -> Connector:Banana_Jack_2Pin
- SW3: value SW_DIP_x01 -> SW_SPDT; footprint Connector:Banana_Jack_2Pin -> Connector_PinHeader_1.27mm:PinHeader_1x03_P1.27mm_Vertical
- U1: footprint Connector_Pin:Pin_D1.3mm_L11.0mm -> Connector_PinHeader_2.54mm:PinHeader_1x10_P2.54mm_Vertical
- moved H4 126.6 mm to (41.0, 125.0)
- moved C7 124.1 mm to (87.0, 192.6)
- moved C5 122.4 mm to (91.1, 191.6)
- moved C6 116.1 mm to (95.5, 185.3)
- moved D7 114.7 mm to (47.0, 173.0)
- moved C16 114.6 mm to (79.0, 191.1)
- moved C9 113.9 mm to (87.1, 187.6)
- moved C8 113.1 mm to (91.1, 186.6)
- moved C11 110.5 mm to (91.4, 184.1)
- moved SW3 106.7 mm to (93.0, 169.8), turned to 0 degrees
- moved H3 106.7 mm to (55.0, 136.0), turned to 0 degrees
- moved C3 106.4 mm to (110.5, 171.9)
- moved C4 103.9 mm to (114.6, 169.4)
- moved C12 100.8 mm to (103.8, 174.4)
- moved C13 100.7 mm to (105.2, 176.9)
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Connections:
- net +12V renamed +24V
- net Net-(D4-Pad1) renamed /StandardizedVRMS/DIODE
- D5 pad 1: +12P -> /StandardizedVRMS/BUCK/V_in
- D6 pad 2: +3V3 -> /StandardizedVRMS/BUCK/V_in
- D7 pad 2: CAN_Shield -> +3V3
- JP1 pad 1: Net-(D7-Pad6) -> Net-(D8-Pad6)
- JP2 pad 1: Net-(D7-Pad4) -> Net-(D8-Pad4)
- JP2 pad 2: /MCU2/CAN1_L -> CAN4_L
- JP3 pad 1: Net-(D7-Pad3) -> Net-(D8-Pad3)
- JP4 pad 1: Net-(D7-Pad1) -> Net-(D8-Pad1)
- R12 pad 1: +12P -> CAN_Shield
- R12 pad 2: Net-(PWR_IN1-Pad2) -> Net-(D6-Pad1)
- R13 pad 2: Net-(PWR_3V1-Pad2) -> /MCU2/I2C1_SCL
- R14 pad 2: /MCU2/I2C1_SCL -> /MCU2/I2C1_SDA
- R15 pad 2: /MCU2/I2C1_SDA -> /MCU2/I2C2_SCL
- R16 pad 2: /MCU2/I2C2_SCL -> /MCU2/I2C2_SDA
- R17 pad 1: +3V3 -> Net-(D7-Pad1)
- R17 pad 2: /MCU2/I2C2_SDA -> CAN_Shield
- R18 pad 1: Net-(D6-Pad1) -> Net-(D9-Pad6)
- R18 pad 2: CAN_Shield -> /MCU2/LED_B
- R19 pad 2: /MCU2/LED_B -> /MCU2/LED_G
- R20 pad 2: /MCU2/LED_G -> /MCU2/LED_R
- R21 pad 1: Net-(D8-Pad4) -> Net-(C13-Pad2)
- R21 pad 2: /MCU2/LED_R -> Net-(D8-Pad4)
- R22 pad 1: Net-(C13-Pad2) -> Net-(C14-Pad2)
- R22 pad 2: Net-(D7-Pad4) -> Net-(D8-Pad1)
- R23 pad 1: Net-(C14-Pad2) -> Net-(C13-Pad2)
- R23 pad 2: Net-(D7-Pad1) -> Net-(D8-Pad4)
- R24 pad 1: Net-(C13-Pad2) -> Net-(C14-Pad2)
- R24 pad 2: Net-(D7-Pad4) -> Net-(D8-Pad1)
- R25 pad 1: Net-(C14-Pad2) -> Net-(D8-Pad6)
- R25 pad 2: Net-(D7-Pad1) -> Net-(J6-Pad2)
- R26 pad 1: Net-(D7-Pad6) -> Net-(D8-Pad3)
- R26 pad 2: Net-(J6-Pad2) -> Net-(J7-Pad2)
- R27 pad 1: Net-(D7-Pad3) -> Net-(D8-Pad6)
- R27 pad 2: Net-(J7-Pad2) -> Net-(J6-Pad2)
- R28 pad 1: Net-(D7-Pad6) -> Net-(D8-Pad3)
- R28 pad 2: Net-(J6-Pad2) -> Net-(J7-Pad2)
- R29 pad 1: Net-(D7-Pad3) -> /MCU2/HSE_out
- R29 pad 2: Net-(J7-Pad2) -> Net-(C16-Pad1)
- R30 pad 1: /MCU2/HSE_out -> Net-(R30-Pad1)
- R30 pad 2: Net-(C16-Pad1) -> /MCU2/BOOT0
- R31 pad 1: Net-(R31-Pad1) -> Net-(J8-Pad2)
- R31 pad 2: /MCU2/BOOT0 -> /MCU2/SWDIO
- SW1 pad 1: +12P -> TSCU_Rst
- SW1 pad 2: VCU_Wake -> CAN_Shield
- SW2 pad 1: TSCU_Rst -> Shutdown_OUT
- SW2 pad 2: TSCU_Rst -> Shutdown_CON
- SW3 pad 1: Shutdown_OUT -> +3V3
- SW3 pad 2: Shutdown_CON -> Net-(R30-Pad1)
- TP10 pad 1: Net-(D7-Pad1) -> Net-(D8-Pad1)
- TP7 pad 1: Net-(D7-Pad6) -> Net-(D8-Pad6)
- TP8 pad 1: Net-(D7-Pad3) -> Net-(D8-Pad3)
- TP9 pad 1: Net-(D7-Pad4) -> Net-(D8-Pad4)
- U2 pad 27: /MCU2/PB1 -> CS
- U3 pad 6: Net-(D7-Pad4) -> Net-(D8-Pad4)
- U3 pad 7: Net-(D7-Pad6) -> Net-(D8-Pad6)
- U4 pad 6: Net-(D7-Pad1) -> Net-(D8-Pad1)
- U4 pad 7: Net-(D7-Pad3) -> Net-(D8-Pad3)
Routing:
- net CAN_Shield: track 101.1 -> 0.00 mm, vias 5 -> 0
- net J1772_Pilot: track 86.4 -> 0.00 mm, vias 2 -> 0
- net J1772_Prox: track 84.9 -> 0.00 mm, vias 2 -> 0
- net Shutdown_OUT: track 56.8 -> 0.00 mm
- net +3V3: track 46.9 -> 0.00 mm, vias 2 -> 0
- net Shutdown_IN: track 37.6 -> 0.00 mm
- net +24V: track 8.33 -> 0.00 mm, vias 1 -> 0
- net Net-(C1-Pad2): track 6.07 -> 0.00 mm
- net +3.3VA: track 5.11 -> 0.00 mm
- net +12P: track 4.83 -> 0.00 mm
Other:
- board outline removed

Commit message: with layout
Parts:
- J1: footprint Connector_PinHeader_2.54mm:PinHeader_1x20_P2.54mm_Vertical -> Connector_Molex:Molex_Micro-Fit_3.0_43045-2010_2x10-1MP_P3.00mm_Horizontal
- moved J2 145.7 mm to (193.0, 81.2), turned to 180 degrees
- moved R31 138.0 mm to (90.9, 56.1), turned to 90 degrees
- moved TP4 132.0 mm to (98.8, 53.6)
- moved TP6 129.5 mm to (101.4, 53.6)
- moved C8 128.9 mm to (105.3, 58.4), turned to -90 degrees
- moved C7 128.9 mm to (106.3, 65.2), turned to -90 degrees
- moved L1 124.1 mm to (100.7, 69.8), turned to 180 degrees
- moved C16 121.0 mm to (97.3, 71.4), turned to 180 degrees
- moved C3 120.6 mm to (93.5, 52.5)
- moved C6 120.6 mm to (104.8, 65.2), turned to -90 degrees
- moved C14 120.5 mm to (109.5, 57.6), turned to 90 degrees
- moved R22 120.1 mm to (110.7, 54.4), turned to 90 degrees
- moved R13 119.9 mm to (80.2, 61.1), turned to 90 degrees
- moved R26 119.9 mm to (109.2, 60.7), turned to -90 degrees
- moved R23 118.1 mm to (109.8, 65.2), turned to 90 degrees
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Routing:
- net CAN_Shield: track 0.00 -> 79.1 mm, vias 0 -> 8
- net +3V3: track 0.00 -> 31.3 mm
- net /MCU2/CAN1_RX: track 0.00 -> 14.7 mm
- net /MCU2/I2C1_SCL: track 0.00 -> 12.8 mm
- net /MCU2/BOOT0: track 0.00 -> 12.6 mm
- net /MCU2/I2C1_SDA: track 0.00 -> 12.1 mm
- net /MCU2/CAN2_TX: track 0.00 -> 10.3 mm
- net Net-(C1-Pad2): track 0.00 -> 10.2 mm
- net Net-(D8-Pad3): track 0.00 -> 9.66 mm
- net /MCU2/CAN1_TX: track 0.00 -> 9.43 mm
- net /MCU2/HSE_in: track 0.00 -> 9.27 mm
- net Net-(C2-Pad2): track 0.00 -> 7.18 mm
- net /StandardizedVRMS/DIODE: track 0.00 -> 6.96 mm
- net CAN3_L: track 0.00 -> 6.62 mm
- net +3.3VA: track 0.00 -> 6.39 mm
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- added copper zone on F.Cu, net +3V3

Commit message: PCB stuff
Parts:
- removed J7: Conn_01x02, Connector_PinHeader_2.54mm:PinHeader_1x02_P2.54mm_Vertical
- moved R24 110.5 mm to (65.7, 81.7), turned to 180 degrees
- moved R27 109.8 mm to (70.1, 80.9), turned to 180 degrees
- moved C5 109.8 mm to (70.2, 83.8)
- moved TP8 109.8 mm to (69.6, 86.5)
- moved R21 109.6 mm to (73.4, 80.9)
- moved TP9 108.9 mm to (72.6, 86.6)
- moved TP3 107.6 mm to (88.2, 83.2)
- moved JP3 100.7 mm to (65.8, 85.4), turned to 180 degrees
- moved J6 98.0 mm to (71.9, 78.0), turned to -90 degrees
- moved JP1 95.8 mm to (76.5, 68.7), turned to 180 degrees
- moved R20 93.8 mm to (93.1, 76.1)
- moved JP4 81.8 mm to (65.6, 78.2)
- moved SW3 81.7 mm to (88.0, 80.3), turned to -90 degrees
- moved JP2 62.8 mm to (75.6, 65.7), turned to 180 degrees
- moved D1 56.9 mm to (78.0, 77.5), turned to 180 degrees
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Routing:
- net CAN_Shield: track 79.1 -> 87.8 mm
- net Net-(D8-Pad3): track 9.66 -> 13.4 mm
- net Net-(D8-Pad1): track 2.18 -> 5.66 mm
- net Net-(C13-Pad2): track 1.82 -> 5.04 mm
- net Net-(D9-Pad4): track 0.00 -> 3.17 mm
- net /MCU2/LED_B: track 0.00 -> 3.04 mm
- net Net-(J6-Pad2): track 0.00 -> 2.96 mm
- net Net-(D1-Pad1): track 0.00 -> 2.16 mm
- net +3V3: track 31.3 -> 32.9 mm

Commit message: new HUD PCB
Parts:
- removed D1: IMD, Dashboard_LED:LEDC1608X80N
- removed D2: AMS, LED_SMD:LED_0805_2012Metric
- removed TP3, TP4: , TestPoint:TestPoint_THTPad_1.0x1.0mm_Drill0.5mm
- added AMS: AMS, LED_SMD:LED_0603_1608Metric, F.Cu at (64.5, 79.4)
- added C17: 10u, Capacitor_SMD:C_0603_1608Metric, F.Cu at (195.1, 61.6)
- added C18: 10u, Capacitor_SMD:C_0603_1608Metric, F.Cu at (193.4, 61.6)
- added C19: 100p, Capacitor_SMD:C_0603_1608Metric, F.Cu at (184.4, 80.2)
- added C20: 10u, Capacitor_SMD:C_0603_1608Metric, F.Cu at (195.2, 58.3)
- added C21: 270p, Capacitor_SMD:C_0603_1608Metric, F.Cu at (176.7, 72.5)
- added C22: 100n, Capacitor_SMD:C_0603_1608Metric, F.Cu at (193.4, 58.3)
- added C23: 220n, Capacitor_SMD:C_0603_1608Metric, F.Cu at (178.9, 83.6)
- added C24: 6.8n, Capacitor_SMD:C_0603_1608Metric, F.Cu at (178.5, 75.8)
- added C25: 1u, Capacitor_SMD:C_0603_1608Metric, F.Cu at (184.2, 75.8)
- added C26: 100p, Capacitor_SMD:C_0603_1608Metric, F.Cu at (182.3, 75.8)
- added C27: 9.4u, Capacitor_SMD:C_0603_1608Metric, F.Cu at (184.2, 72.4)
- added C28: 66u, Capacitor_SMD:C_0603_1608Metric, F.Cu at (187.9, 35.1)
- added C29: 10uF, Capacitor_SMD:C_0603_1608Metric_Pad1.08x0.95mm_HandSolder, F.Cu at (167.0, 70.8)
- added C30: 10uF, Capacitor_SMD:C_0603_1608Metric_Pad1.08x0.95mm_HandSolder, F.Cu at (167.0, 74.5)
- added C31: 100nF, Capacitor_SMD:C_0603_1608Metric_Pad1.08x0.95mm_HandSolder, F.Cu at (167.0, 72.5)
- added C32: 100nF, Capacitor_SMD:C_0603_1608Metric_Pad1.08x0.95mm_HandSolder, F.Cu at (167.1, 63.2)
- added C33: 22uF, Capacitor_SMD:C_0603_1608Metric_Pad1.08x0.95mm_HandSolder, F.Cu at (171.0, 63.6)
- added C34: 22uF, Capacitor_SMD:C_0603_1608Metric_Pad1.08x0.95mm_HandSolder, F.Cu at (171.0, 65.5)
- added C35: 1uF, Capacitor_SMD:C_0603_1608Metric_Pad1.08x0.95mm_HandSolder, F.Cu at (171.0, 61.6)
- added C36: 22uF, Capacitor_SMD:C_0603_1608Metric_Pad1.08x0.95mm_HandSolder, F.Cu at (167.1, 61.3)
- added D10: STPS20M100SG-TR, Global Libraries_2:STPS20M100SG-TR, F.Cu at (186.2, 44.7)
- added D8: DT1446-04TS-7, Global Libraries_2:SOT95P280X100-6N, F.Cu at (95.0, 50.1)
- added IC1: LM5155DSSR, Global Libraries_2:SON50P200X300X80-13N-D, F.Cu at (179.6, 80.1)
- added IMD: IMD, Dashboard_LED:LEDC1608X80N, F.Cu at (61.7, 79.4)
- added J7: Conn_01x02, Connector_PinHeader_2.54mm:PinHeader_1x02_P2.54mm_Vertical, F.Cu at (106.4, 51.5)
- added JP5: , Jumper:SolderJumper-2_P1.3mm_Bridged2Bar_Pad1.0x1.5mm, F.Cu at (73.6, 68.8)
- added JP6: , Jumper:SolderJumper-2_P1.3mm_Bridged2Bar_Pad1.0x1.5mm, F.Cu at (73.5, 65.6)
- added JP7: , Jumper:SolderJumper-2_P1.3mm_Bridged2Bar_Pad1.0x1.5mm, F.Cu at (98.4, 49.2)
- added JP8: , Jumper:SolderJumper-2_P1.3mm_Bridged2Bar_Pad1.0x1.5mm, F.Cu at (111.6, 55.9)
- added L2: 7448700015, Inductor Thing:WE-DD_12XX_CROSSED12, F.Cu at (185.9, 63.2)
- added L3: 4u7, Inductor_SMD:L_Sunlord_MWSA0518_5.4x5.2mm, F.Cu at (161.4, 65.9)
- added Q1: CSD18537NQ5A, Global Libraries_2:CSD19531Q5AT, F.Cu at (189.9, 74.3)
- added R32: 6k8, Resistor_SMD:R_0603_1608Metric, F.Cu at (186.3, 80.2)
- added R33: 34k8, Resistor_SMD:R_0603_1608Metric, F.Cu at (182.5, 80.2)
- added R34: 17k8, Resistor_SMD:R_0603_1608Metric, F.Cu at (180.7, 83.6)
- added R35: 10k, Resistor_SMD:R_0603_1608Metric, F.Cu at (178.6, 72.4)
- added R36: 100, Resistor_SMD:R_0603_1608Metric, F.Cu at (180.5, 75.7)
- added R37: 4m, Resistor_SMD:R_0603_1608Metric, F.Cu at (182.3, 72.4)
- added R38: 4m, Resistor_SMD:R_0603_1608Metric, F.Cu at (180.5, 72.4)
- added R39: 51k1, Resistor_SMD:R_0603_1608Metric, F.Cu at (187.8, 36.9)
- added R40: 4k7, Resistor_SMD:R_0603_1608Metric, F.Cu at (184.5, 36.9)
- added R41: 10K, Resistor_SMD:R_0603_1608Metric_Pad0.98x0.95mm_HandSolder, F.Cu at (167.0, 68.9)
- added R42: 10K, Resistor_SMD:R_0603_1608Metric_Pad0.98x0.95mm_HandSolder, F.Cu at (170.6, 70.8)
- added R43: 54.9K, Resistor_SMD:R_0603_1608Metric_Pad0.98x0.95mm_HandSolder, F.Cu at (170.5, 68.9)
- added TP1: , TestPoint:TestPoint_THTPad_1.0x1.0mm_Drill0.5mm, F.Cu at (78.5, 72.3)
- added TP11: , TestPoint:TestPoint_THTPad_1.0x1.0mm_Drill0.5mm, F.Cu at (78.5, 69.2)
- added TP12: , TestPoint:TestPoint_THTPad_1.0x1.0mm_Drill0.5mm, F.Cu at (98.4, 52.3)
- added TP13: , TestPoint:TestPoint_THTPad_1.0x1.0mm_Drill0.5mm, F.Cu at (76.4, 63.0)
- added TP14: , TestPoint:TestPoint_THTPad_1.0x1.0mm_Drill0.5mm, F.Cu at (108.5, 55.9)
- added TP2: , TestPoint:TestPoint_THTPad_1.0x1.0mm_Drill0.5mm, F.Cu at (76.9, 81.9)
- added U5: LMR51420, Package_TO_SOT_SMD:SOT-23-6, F.Cu at (167.1, 66.0)
- added U6: AMS1117-3.3, Package_TO_SOT_SMD:SOT-223-3_TabPin2, F.Cu at (168.4, 55.8)
- Pilot TP: renamed from TP1
- Prox TP: renamed from TP2
- SW2: footprint Connector:Banana_Jack_2Pin -> Connector_Wire:SolderWire-0.1sqmm_1x02_P3.6mm_D0.4mm_OD1mm
- moved H3 173.4 mm to (194.1, 32.4)
- moved H4 157.3 mm to (194.1, 88.5)
- moved J2 112.1 mm to (88.9, 39.5)
- moved SW2 109.0 mm to (68.9, 57.0), turned to -90 degrees
- moved F1 106.2 mm to (188.8, 80.8), turned to 90 degrees
- moved D5 102.8 mm to (185.3, 86.0)
- moved D4 98.7 mm to (185.7, 82.9), turned to 180 degrees
- moved D3 97.1 mm to (171.5, 49.3), turned to 90 degrees
- moved R3 96.6 mm to (174.4, 50.2)
- moved S1 85.7 mm to (171.5, 45.7)
- moved D6 84.1 mm to (163.2, 74.5), turned to 0 degrees
- moved R12 81.5 mm to (163.2, 76.8)
- moved H1 76.8 mm to (50.7, 33.3)
- moved R24 45.7 mm to (102.9, 55.1), turned to 90 degrees
- moved TP8 39.0 mm to (95.0, 56.9)
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Connections:
- J1 pad 1: Shutdown_IN -> IMD_LED
- J1 pad 10: CAN1_H -> J1772_Pilot
- J1 pad 11: CAN1_L -> AMS_LED
- J1 pad 12: CAN2_H -> CAN2_L
- J1 pad 13: CAN2_L -> CAN4_H
- J1 pad 14: CAN3_H -> Shutdown_IN
- J1 pad 15: CAN3_L -> Shutdown_CON
- J1 pad 16: CAN4_H -> Shutdown_OUT
- J1 pad 17: CAN4_L -> CAN3_H
- J1 pad 18: CAN_Shield -> TSCU_Rst
- J1 pad 19: VCU_Wake -> CAN1_L
- J1 pad 2: Shutdown_OUT -> CAN2_H
- J1 pad 20: TSCU_Rst -> J1772_Prox
- J1 pad 3: Shutdown_CON -> CAN4_L
- J1 pad 6: AMS_LED -> CAN_Shield
- J1 pad 7: IMD_LED -> CAN3_L
- J1 pad 8: J1772_Pilot -> VCU_Wake
- J1 pad 9: J1772_Prox -> CAN1_H
- J4 pad 1: Net-(C2-Pad2) -> Shutdown_IN
- J4 pad 2: Net-(J4-Pad2) -> Shutdown_CON
- J5 pad 1: Shutdown_IN -> Net-(C2-Pad2)
- J5 pad 2: Shutdown_CON -> Net-(J5-Pad2)
- JP1 pad 1: Net-(D8-Pad6) -> Net-(JP1-Pad1)
- JP1 pad 2: CAN4_H -> CAN2_H
- JP2 pad 1: Net-(D8-Pad4) -> Net-(JP2-Pad1)
- JP2 pad 2: CAN4_L -> CAN2_L
- JP3 pad 1: Net-(D8-Pad3) -> Net-(JP3-Pad1)
- JP3 pad 2: /MCU2/CAN2_H -> CAN3_H
- JP4 pad 1: Net-(D8-Pad1) -> Net-(JP4-Pad1)
- JP4 pad 2: /MCU2/CAN2_L -> CAN3_L
- R10 pad 1: CAN2_H -> Net-(JP3-Pad1)
- R10 pad 2: Net-(J3-Pad2) -> Net-(J5-Pad2)
- R11 pad 1: CAN3_H -> Net-(JP3-Pad1)
- R11 pad 2: Net-(J4-Pad2) -> Net-(J5-Pad2)
- R4 pad 2: CAN2_L -> Net-(JP2-Pad1)
- R5 pad 1: Net-(C2-Pad2) -> Net-(C1-Pad2)
- R5 pad 2: CAN3_L -> Net-(JP2-Pad1)
- R6 pad 1: Net-(C1-Pad2) -> Net-(JP1-Pad1)
- R6 pad 2: CAN2_L -> Net-(J3-Pad2)
- R7 pad 1: Net-(C2-Pad2) -> Net-(JP1-Pad1)
- R7 pad 2: CAN3_L -> Net-(J3-Pad2)
- R8 pad 1: CAN2_H -> Net-(C2-Pad2)
- R8 pad 2: Net-(J3-Pad2) -> Net-(JP4-Pad1)
- R9 pad 1: CAN3_H -> Net-(C2-Pad2)
- R9 pad 2: Net-(J4-Pad2) -> Net-(JP4-Pad1)
- TP10 pad 1: Net-(D8-Pad1) -> /MCU2/CAN2_RX
- TP5 pad 1: /MCU2/CAN1_RX -> Net-(JP3-Pad1)
- TP6 pad 1: /MCU2/CAN2_RX -> Net-(JP4-Pad1)
- TP7 pad 1: Net-(D8-Pad6) -> /MCU2/CAN1_TX
- TP8 pad 1: Net-(D8-Pad3) -> /MCU2/CAN2_TX
- TP9 pad 1: Net-(D8-Pad4) -> /MCU2/CAN1_RX
Routing:
- net +24V: track 0.00 -> 206.9 mm, vias 0 -> 2
- net +3V3: track 32.9 -> 160.3 mm, vias 0 -> 3
- net +5V: track 0.00 -> 123.1 mm, vias 0 -> 3
- net VCU_Wake: track 0.00 -> 119.4 mm
- net /SEPIC_CAD/FB: track 0.00 -> 57.9 mm
- net CS: track 0.00 -> 48.0 mm
- net Net-(D8-Pad4): track 0.00 -> 46.5 mm
- net D/C: track 0.00 -> 45.2 mm
- net CAN_Shield: track 87.8 -> 130.2 mm, vias 8 -> 45
- net CAN1_H: track 0.00 -> 38.2 mm
- net MOSI: track 0.00 -> 37.0 mm
- net /StandardizedVRMS/BUCK/V_in: track 0.00 -> 35.9 mm
- net Net-(D8-Pad6): track 3.68 -> 38.4 mm
- net SCK: track 0.00 -> 34.0 mm
- net +12V: track 0.00 -> 33.7 mm
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- added copper zone on B.Cu, net CAN_Shield
- added copper zone on F.Cu, net CAN_Shield
- removed copper zone on F.Cu, net +3V3
Other:
- board outline added: 152.5 x 64.6 mm

Commit message: revisions
Routing:
- net CAN_Shield: track 130.2 -> 147.3 mm, vias 45 -> 46
Changed lines of the file:
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@@
     (property "Sheetname" "MCU2")
     (attr smd)
-    (fp_text reference "C13" (at 0.1 1.5656) (layer "F.SilkS")
+    (fp_text reference "C13" (at -0.5096 1.5656) (layer "F.SilkS")
       (effects (font (size 1 1) (thickness 0.15)))
     )
@@
   (segment (start 96.3908 79.6452) (end 96.3908 77.8672) (width 0.25) (layer "F.Cu") (net 1))
   (segment (start 86.0406 69.1804) (end 85.663849 69.1804) (width 0.25) (layer "F.Cu") (net 1))
+  (segment (start 95.0518 53.599) (end 95.3932 53.9404) (width 0.25) (layer "F.Cu") (net 1))
   (segment (start 64.3514 83.692) (end 64.4144 83.629) (width 0.25) (layer "F.Cu") (net 1))
   (segment (start 167.8929 70.8163) (end 167.841 70.7644) (width 0.25) (layer "F.Cu") (net 1))
@@
   (segment (start 92.048 60.646) (end 92.048 58.881) (width 0.25) (layer "F.Cu") (net 1))
   (segment (start 86.3323 74.7173) (end 85.5323 73.9173) (width 0.25) (layer "F.Cu") (net 1))
+  (segment (start 86.8172 78.994) (end 84.1756 78.994) (width 0.25) (layer "F.Cu") (net 1))
   (segment (start 89.662 75.2986) (end 88.8438 75.2986) (width 0.25) (layer "F.Cu") (net 1))
   (segment (start 97.4934 75.1526) (end 97.4934 73.9918) (width 0.25) (layer "F.Cu") (net 1))
@@
   (segment (start 185.4826 35.0744) (end 187.0944 35.0744) (width 0.25) (layer "F.Cu") (net 1))
   (segment (start 193.4196 62.367) (end 195.1338 62.367) (width 0.25) (layer "F.Cu") (net 1))
+  (segment (start 81.961 59.2836) (end 81.026 59.2836) (width 0.25) (layer "F.Cu") (net 1))
   (segment (start 167.229 62.2796) (end 169.5219 62.2796) (width 0.25) (layer "F.Cu") (net 1))
   (segment (start 92.048 58.881) (end 92.035 58.868) (width 0.25) (layer "F.Cu") (net 1))
@@
   (segment (start 169.5219 62.2796) (end 170.1811 61.6204) (width 0.25) (layer "F.Cu") (net 1))
   (segment (start 85.663849 69.1804) (end 84.7406 70.103649) (width 0.25) (layer "F.Cu") (net 1))
+  (segment (start 92.1666 53.599) (end 95.0518 53.599) (width 0.25) (layer "F.Cu") (net 1))
   (segment (start 96.2738 53.9404) (end 95.3932 53.9404) (width 0.25) (layer "F.Cu") (net 1))
   (segment (start 95.818 50.0796) (end 96.3114 50.0796) (width 0.25) (layer "F.Cu") (net 1))
+  (segment (start 84.1756 78.994) (end 81.2292 81.9404) (width 0.25) (layer "F.Cu") (net 1))
   (segment (start 105.096 64.5706) (end 105.1052 64.5798) (width 0.25) (layer "F.Cu") (net 1))
   (segment (start 96.3908 77.8672) (end 97.1153 77.1427) (width 0.25) (layer "F.Cu") (net 1))
@@
   (segment (start 61.722 83.692) (end 64.3514 83.692) (width 0.25) (layer "F.Cu") (net 1))
   (segment (start 191.516 56.4896) (end 196.2404 56.4896) (width 0.25) (layer "F.Cu") (net 1))
+  (segment (start 87.7916 78.0196) (end 86.8172 78.994) (width 0.25) (layer "F.Cu") (net 1))
+  (segment (start 83.425 60.7476) (end 81.961 59.2836) (width 0.25) (layer "F.Cu") (net 1))
   (segment (start 86.3323 74.7173) (end 87.8827 74.7173) (width 0.25) (layer "F.Cu") (net 1))
   (segment (start 195.1716 62.38) (end 195.1468 62.38) (width 0.25) (layer "F.Cu") (net 1))
   (segment (start 196.2404 58.073) (end 195.1976 59.1158) (width 0.25) (layer "F.Cu") (net 1))
   (segment (start 92.883 81.5484) (end 92.883 80.0088) (width 0.25) (layer "F.Cu") (net 1))
+  (segment (start 90.3938 78.0196) (end 87.7916 78.0196) (width 0.25) (layer "F.Cu") (net 1))
   (segment (start 167.8918 70.8152) (end 167.841 70.7644) (width 0.25) (layer "F.Cu") (net 1))
   (segment (start 190.1952 57.8104) (end 191.516 56.4896) (width 0.25) (layer "F.Cu") (net 1))
@@
   (via (at 56.388 64.2112) (size 0.8) (drill 0.4) (layers "F.Cu" "B.Cu") (free) (net 1))
   (via (at 163.2712 59.6392) (size 0.8) (drill 0.4) (layers "F.Cu" "B.Cu") (free) (net 1))
+  (via (at 81.026 59.2836) (size 0.8) (drill 0.4) (layers "F.Cu" "B.Cu") (net 1))
   (via (at 163.2712 58.674) (size 0.8) (drill 0.4) (layers "F.Cu" "B.Cu") (free) (net 1))
   (via (at 164.592 78.994) (size 0.8) (drill 0.4) (layers "F.Cu" "B.Cu") (free) (net 1))
